File: matrix.kicad_sch (KiCad schematic)
At the start: 146 parts

Commit message: add PCB
Parts:
- D1, D10, D11, D12, D13, D14, D15, D16, D17, D18, D19, D2, D20, D21, D22, D23, D24, D25, D26, D27, D28, D29, D3, D30, D31, D32, D33, D34, D35, D36, D37, D38, D39, D4, D40, D41, D42, D43, D44, D45, D46, D47, D48, D49, D5, D50, D51, D52, D53, D54, D55, D56, D57, D58, D59, D6, D60, D61, D62, D63, D7, D8, D9: footprint (none) -> Diode_SMD:D_SOD-123
Connections:
- net COL00: now also MX31.2; no longer MX31.1, MX45.1
- net COL01: now also MX2.2, MX45.2, MX60.2, MX68.2; no longer MX2.1, MX60.1, MX68.1
- net COL02: now also MX3.2, MX46.2; no longer MX3.1, MX46.1
- net COL03: now also MX4.2, MX47.2; no longer MX4.1, MX47.1
- net COL04: now also MX48.2, MX5.2; no longer MX48.1, MX5.1
- net COL05: now also MX49.2, MX6.2; no longer MX49.1, MX6.1
- net COL06: now also MX50.2, MX7.2; no longer MX50.1, MX7.1
- net COL07: now also MX51.2, MX8.2; no longer MX51.1, MX8.1
- net COL08: now also MX52.2, MX9.2; no longer MX52.1, MX9.1
- net COL09: now also MX10.2, MX53.2; no longer MX10.1, MX53.1
- net COL10: now also MX11.2, MX54.2; no longer MX11.1, MX54.1
- net COL11: now also MX12.2, MX55.2; no longer MX12.1, MX55.1
- net COL12: now also MX13.2, MX28.2, MX43.2, MX65.2, MX72.2; no longer MX13.1, MX28.1, MX43.1, MX65.1, MX72.1
- net COL13: now also MX14.2, MX57.2, MX66.2, MX73.2; no longer MX14.1, MX57.1, MX66.1, MX73.1
- net ROW2: no longer D29.1 (K)
- net ROW3: now also D29.1 (K)
- net at D3.2 (A): now also MX3.1; no longer MX3.2
- net at D53.2 (A): now also MX55.1; no longer MX55.2
- net at D29.2 (A), MX30.2: now also MX31.1; no longer MX31.2
- net at D51.2 (A): now also MX53.1; no longer MX53.2
- net at D9.2 (A): now also MX9.1; no longer MX9.2
- net at D7.2 (A): now also MX7.1; no longer MX7.2
- net at D44.2 (A): now also MX46.1; no longer MX46.2
- net at D55.2 (A): now also MX57.1; no longer MX57.2
- net at D6.2 (A): now also MX6.1; no longer MX6.2
- net at D50.2 (A): now also MX52.1; no longer MX52.2
- net at D27.2 (A): now also MX28.1; no longer MX28.2
- net at D12.2 (A): now also MX12.1; no longer MX12.2
- net at D43.2 (A): now also MX45.1; no longer MX45.2
- net at D48.2 (A): now also MX50.1; no longer MX50.2
- net at D2.2 (A): now also MX2.1; no longer MX2.2
- net at D46.2 (A): now also MX48.1; no longer MX48.2
- net at D11.2 (A): now also MX11.1; no longer MX11.2
- net at D41.2 (A): now also MX43.1; no longer MX43.2
- net at D52.2 (A): now also MX54.1; no longer MX54.2
- net at D14.2 (A), MX15.2: now also MX14.1; no longer MX14.2
- net at D5.2 (A): now also MX5.1; no longer MX5.2
- net at D10.2 (A): now also MX10.1; no longer MX10.2
- net at D8.2 (A): now also MX8.1; no longer MX8.2
- net at D45.2 (A): now also MX47.1; no longer MX47.2
- net at D49.2 (A): now also MX51.1; no longer MX51.2
- net at D4.2 (A): now also MX4.1; no longer MX4.2
- net at D47.2 (A): now also MX49.1; no longer MX49.2
- net at D13.2 (A): now also MX13.1; no longer MX13.2
- new net: D62.2 (A), MX65.1, MX72.1
- new net: D63.2 (A), MX66.1, MX73.1
- new net: D57.2 (A), MX60.1, MX68.1
Other:
- moved on the sheet: D29, D43, MX10, MX11, MX12, MX13, MX14, MX2, MX28, MX3, MX30, MX31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
